File: doc/pcb/LEDnode/LEDnode.kicad_sch (KiCad schematic)
At the start: 72 parts, among them J1 Ni-MH, J2 SWD, J3 GPIO1, J4 GPIO2, Q1 PDTB113ET.215, Q2 PDTB113ET.215, Q3 PDTB113ET.215, Q4 PDTB113ET.215, Q5 IRLML6346, Q6 BSS138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

Commit message: new pcb
Parts:
- added C21, C22: 476, Capacitor_SMD:CP_Elec_5x4.5, symbol Device:C_Polarized
- added H5: Copy Number, BartLib_Logo:number, symbol Mechanical:MountingHole_Pad
- added Q7: IRLML6346, Package_TO_SOT_SMD:SOT-23, symbol Device:Q_NMOS_GSD
- added R26: 100k, Resistor_SMD:R_0603_1608Metric, symbol Device:R
- added R27: 0, Resistor_SMD:R_0603_1608Metric, symbol Device:R
- SW3: value TL3342F160QG -> 6x6 13; footprint Button_Switch_SMD:SW_SPST_B3SL-1002P -> Button_Switch_THT:SW_PUSH_6mm_H13mm
Connections:
- net +3V3: now also C22.1, R26.1
- net GND: now also C21.2, C22.2, Q7.3 (D)
- net INPUT: now also C21.1, Q7.1 (G), R27.1; no longer U1.7 (PA0)
- new net BACKUP: Q7.2 (S), R26.2, R27.2, U1.7 (PA0)
- no-connect marks 3 -> 4
Other:
- note added: "Q6,R8-Encoder control by MCU / R13-force active"
- note added: "Q7,R26,C22-EXTI backup system / R27, C21-power backup"
- moved on the sheet: C2, C3, C6, C7
