File: doc/pcb/Mk2/LEDnode/LEDnode.kicad_pcb (KiCad board)
At the start: 2 copper layers, 55 x 36.5 mm, 76 parts, among them J1 Ni-MH, J2 SWD, J4 GPIO2, Q1 PDTB113ET.215, Q2 PDTB113ET.215, Q3 PDTB113ET.215, Q4 PDTB113ET.215, Q5 IRLML6346, Q6 BSS138, Q7 IRLML6346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

Commit message: corrected backup transistor
Parts:
- C21: value 500m_SE-5R5-D224VYH3E -> 220mF_SE-5R5-D224VYH3E
Connections:
- Q7 pad 2: /BACKUP -> GND
- Q7 pad 3: GND -> /BACKUP
Routing:
- net /BACKUP: track 24.9 -> 27.3 mm
- net /SCL: track 93.1 -> 91.7 mm
Other:
- board text added: "v1.1"
- board text removed: "v1.0"
Changed lines of the file:
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@@
       (effects (font (size 1 1) (thickness 0.15)))
     )
-    (fp_text value "500m_SE-5R5-D224VYH3E" (at 0 -7.39 180 unlocked) (layer "F.Fab")
+    (fp_text value "220mF_SE-5R5-D224VYH3E" (at 0 -7.39 180 unlocked) (layer "F.Fab")
       (effects (font (size 1 1) (thickness 0.15)))
     )
@@
       (net 1 "/INPUT") (pinfunction "G") (pintype "input"))
     (pad "2" smd roundrect (at -0.9375 -0.95) (size 1.475 0.6) (layers "B.Cu" "B.Paste" "B.Mask") (roundrect_rratio 0.25)
-      (net 53 "/BACKUP") (pinfunction "S") (pintype "passive"))
+      (net 2 "GND") (pinfunction "S") (pintype "passive"))
     (pad "3" smd roundrect (at 0.9375 0) (size 1.475 0.6) (layers "B.Cu" "B.Paste" "B.Mask") (roundrect_rratio 0.25)
-      (net 2 "GND") (pinfunction "D") (pintype "passive"))
+      (net 53 "/BACKUP") (pinfunction "D") (pintype "passive"))
     (model "${KICAD6_3DMODEL_DIR}/Package_TO_SOT_SMD.3dshapes/SOT-23.wrl"
       (offset (xyz 0 0 0))
@@
     (effects (font (size 1 1) (thickness 0.15) italic) (justify left mirror))
   )
-  (gr_text "v1.0" (at 106.9 104) (layer "F.SilkS")
+  (gr_text "v1.1" (at 106.9 104) (layer "F.SilkS")
     (effects (font (size 0.7 0.7) (thickness 0.15)))
   )
@@
   (segment (start 113 88) (end 113.75 87.25) (width 0.25) (layer "F.Cu") (net 16))
   (segment (start 105.6 89) (end 105.774511 89.174511) (width 0.25) (layer "F.Cu") (net 16))
-  (segment (start 81.7 79.9255) (end 81.31275 80.31275) (width 0.25) (layer "F.Cu") (net 16))
   (segment (start 110.5 78) (end 110.5 77.862989) (width 0.25) (layer "F.Cu") (net 16))
   (segment (start 111.5 88) (end 113 88) (width 0.25) (layer "F.Cu") (net 16))
   (segment (start 101.285489 91.748533) (end 101.285489 89.190489) (width 0.25) (layer "F.Cu") (net 16))
   (segment (start 99.45 93.5) (end 99.575 93.5) (width 0.25) (layer "F.Cu") (net 16))
+  (segment (start 86.520607 76.274511) (end 89.625489 76.274511) (width 0.25) (layer "F.Cu") (net 16))
   (segment (start 99.575 93.5) (end 99.675 93.6) (width 0.25) (layer "F.Cu") (net 16))
-  (segment (start 76.62502 75.325958) (end 76.62502 76.42502) (width 0.25) (layer "F.Cu") (net 16))
+  (segment (start 80.624511 72.575489) (end 84.347085 72.575489) (width 0.25) (layer "F.Cu") (net 16))
+  (segment (start 84.347085 72.575489) (end 86.125489 74.353893) (width 0.25) (layer "F.Cu") (net 16))
   (segment (start 110.5 77.862989) (end 109.287011 76.65) (width 0.25) (layer "F.Cu") (net 16))
-  (segment (start 81.7 79.246096) (end 81.7 79.9255) (width 0.25) (layer "F.Cu") (net 16))
+  (segment (start 86.125489 75.879393) (end 86.520607 76.274511) (width 0.25) (layer "F.Cu") (net 16))
+  (segment (start 89.625489 76.274511) (end 93.2 72.7) (width 0.25) (layer "F.Cu") (net 16))
+  (segment (start 77.175489 74.775489) (end 78.424511 74.775489) (width 0.25) (layer "F.Cu") (net 16))
   (segment (start 101.201467 91.748533) (end 99.45 93.5) (width 0.25) (layer "F.Cu") (net 16))
-  (segment (start 109.287011 76.65) (end 109.287011 76.15) (width 0.25) (layer "F.Cu") (net 16))
-  (segment (start 77.175489 74.775489) (end 76.62502 75.325958) (width 0.25) (layer "F.Cu") (net 16))
+  (segment (start 76.62502 76.42502) (end 76.62502 75.325958) (width 0.25) (layer "F.Cu") (net 16))
   (segment (start 108.075489 89.174511) (end 108.125 89.125) (width 0.25) (layer "F.Cu") (net 16))
-  (segment (start 105.837011 72.7) (end 93.2 72.7) (width 0.25) (layer "F.Cu") (net 16))
+  (segment (start 78.424511 74.775489) (end 80.624511 72.575489) (width 0.25) (layer "F.Cu") (net 16))
   (segment (start 108.125 89.125) (end 110.375 89.125) (width 0.25) (layer "F.Cu") (net 16))
-  (segment (start 93.2 72.7) (end 88.575489 77.324511) (width 0.25) (layer "F.Cu") (net 16))
+  (segment (start 77.515489 77.315489) (end 76.62502 76.42502) (width 0.25) (layer "F.Cu") (net 16))
+  (segment (start 86.125489 74.353893) (end 86.125489 75.879393) (width 0.25) (layer "F.Cu") (net 16))
+  (segment (start 76.62502 75.325958) (end 77.175489 74.775489) (width 0.25) (layer "F.Cu") (net 16))
   (segment (start 80.327289 82.6875) (end 79.1325 82.6875) (width 0.25) (layer "F.Cu") (net 16))
+  (segment (start 81.7 79.246096) (end 79.769393 77.315489) (width 0.25) (layer "F.Cu") (net 16))
+  (segment (start 93.2 72.7) (end 105.837011 72.7) (width 0.25) (layer "F.Cu") (net 16))
   (segment (start 105.774511 89.174511) (end 108.075489 89.174511) (width 0.25) (layer "F.Cu") (net 16))
+  (segment (start 109.287011 76.15) (end 109.287011 76.65) (width 0.25) (layer "F.Cu") (net 16))
   (segment (start 114.5 87) (end 114.5 84.5) (width 0.25) (layer "F.Cu") (net 16))
-  (segment (start 84.347085 72.575489) (end 80.624511 72.575489) (width 0.25) (layer "F.Cu") (net 16))
   (segment (start 113.75 87.25) (end 114.25 87.25) (width 0.25) (layer "F.Cu") (net 16))
-  (segment (start 80.624511 72.575489) (end 78.424511 74.775489) (width 0.25) (layer "F.Cu") (net 16))
+  (segment (start 81.1255 80.5) (end 81.7 79.9255) (width 0.25) (layer "F.Cu") (net 16))
   (segment (start 101.285489 89.190489) (end 101.475978 89) (width 0.25) (layer "F.Cu") (net 16))
   (segment (start 101.475978 89) (end 105.6 89) (width 0.25) (layer "F.Cu") (net 16))
-  (segment (start 76.62502 76.42502) (end 77.515489 77.315489) (width 0.25) (layer "F.Cu") (net 16))
-  (segment (start 79.769393 77.315489) (end 81.7 79.246096) (width 0.25) (layer "F.Cu") (net 16))
-  (segment (start 78.424511 74.775489) (end 77.175489 74.775489) (width 0.25) (layer "F.Cu") (net 16))
   (segment (start 114.25 87.25) (end 114.5 87) (width 0.25) (layer "F.Cu") (net 16))
+  (segment (start 79.769393 77.315489) (end 77.515489 77.315489) (width 0.25) (layer "F.Cu") (net 16))
   (segment (start 79.1325 82.6875) (end 78.3 83.52) (width 0.25) (layer "F.Cu") (net 16))
-  (segment (start 81.1255 80.5) (end 81.31275 80.31275) (width 0.25) (layer "F.Cu") (net 16))
-  (segment (start 86.675489 77.324511) (end 86.125489 76.774511) (width 0.25) (layer "F.Cu") (net 16))
-  (segment (start 77.515489 77.315489) (end 79.769393 77.315489) (width 0.25) (layer "F.Cu") (net 16))
-  (segment (start 109.287011 76.15) (end 105.837011 72.7) (width 0.25) (layer "F.Cu") (net 16))
-  (segment (start 86.125489 74.353893) (end 84.347085 72.575489) (width 0.25) (layer "F.Cu") (net 16))
+  (segment (start 81.7 79.9255) (end 81.7 79.246096) (width 0.25) (layer "F.Cu") (net 16))
+  (segment (start 105.837011 72.7) (end 109.287011 76.15) (width 0.25) (layer "F.Cu") (net 16))
   (segment (start 101.285489 91.748533) (end 101.201467 91.748533) (width 0.25) (layer "F.Cu") (net 16))
-  (segment (start 86.125489 76.774511) (end 86.125489 74.353893) (width 0.25) (layer "F.Cu") (net 16))
   (segment (start 110.375 89.125) (end 111.5 88) (width 0.25) (layer "F.Cu") (net 16))
-  (segment (start 88.575489 77.324511) (end 86.675489 77.324511) (width 0.25) (layer "F.Cu") (net 16))
   (via (at 114.5 84.5) (size 0.8) (drill 0.4) (layers "F.Cu" "B.Cu") (net 16))
   (via (at 110.5 78) (size 0.8) (drill 0.4) (layers "F.Cu" "B.Cu") (net 16))
@@
   (segment (start 95.197879 78.102121) (end 95.75 77.55) (width 0.25) (layer "B.Cu") (net 52))
   (segment (start 95.197879 82.569452) (end 95.197879 78.102121) (width 0.25) (layer "B.Cu") (net 52))
-  (segment (start 84.5125 76.65) (end 85.0125 76.15) (width 0.25) (layer "F.Cu") (net 53))
-  (segment (start 81.55 76.65) (end 84.5125 76.65) (width 0.25) (layer "F.Cu") (net 53))
+  (segment (start 85.339244 76.65) (end 85.789244 77.1) (width 0.25) (layer "F.Cu") (net 53))
+  (segment (start 85.789244 77.1) (end 86.8875 77.1) (width 0.25) (layer "F.Cu") (net 53))
+  (segment (start 85.339244 76.65) (end 81.55 76.65) (width 0.25) (layer "F.Cu") (net 53))
   (via (at 81.55 76.65) (size 0.8) (drill 0.4) (layers "F.Cu" "B.Cu") (net 53))
-  (via (at 85.0125 76.15) (size 0.8) (drill 0.4) (layers "F.Cu" "B.Cu") (net 53))
+  (via (at 86.8875 77.1) (size 0.8) (drill 0.4) (layers "F.Cu" "B.Cu") (net 53))
   (segment (start 83.15 79.425) (end 83.125 79.425) (width 0.25) (layer "B.Cu") (net 53))
   (segment (start 85.898945 86.998945) (end 86.226055 87.326055) (width 0.25) (layer "B.Cu") (net 53))
   (segment (start 82.473945 80.076055) (end 85.898945 83.501055) (width 0.25) (layer "B.Cu") (net 53))
   (segment (start 81.85 76.65) (end 81.55 76.65) (width 0.25) (layer "B.Cu") (net 53))
+  (segment (start 86.8875 77.1) (end 86.4 77.1) (width 0.25) (layer "B.Cu") (net 53))
   (segment (start 82.2 77) (end 81.85 76.65) (width 0.25) (layer "B.Cu") (net 53))
   (segment (start 90.7 88.45) (end 90.7 88.30211) (width 0.25) (layer "B.Cu") (net 53))

Commit message: 1.4
Parts:
- Q7: value IRLML6346 -> BSS138
Changed lines of the file:
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@@
       (effects (font (size 1 1) (thickness 0.15)))
     )
-    (fp_text user "LR03 1,2V Ni-MH" (at 0.75 -0.5 unlocked) (layer "F.SilkS")
+    (fp_text user "LR03 1.2V Ni-MH" (at 0.75 -0.5 unlocked) (layer "F.SilkS")
       (effects (font (size 1 1) (thickness 0.15)))
     )
@@
       (effects (font (size 1 1) (thickness 0.15)) (justify mirror))
     )
-    (fp_text value "IRLML6346" (at 0 -2.4) (layer "B.Fab")
+    (fp_text value "BSS138" (at 0 -2.4) (layer "B.Fab")
       (effects (font (size 1 1) (thickness 0.15)) (justify mirror))
     )
@@
   (gr_arc (start 131.5 103.5) (mid 131.06066 104.56066) (end 130 105) (layer "Edge.Cuts") (width 0.1))
   (gr_line (start 104 68.5) (end 130 68.5) (layer "Edge.Cuts") (width 0.1))
-  (gr_line (start 148.001903 74.448097) (end 148.001903 99.051903) (layer "User.2") (width 2.1))
-  (gr_line (start 58.924048 99.052855) (end 58.924048 74.449049) (layer "User.2") (width 2.1))
-  (gr_line (start 190.000001 14.390001) (end 190.000001 17.950001) (layer "User.2") (width 0.05))
-  (gr_line (start 222.5 12) (end 221.99504 14.395629) (layer "User.2") (width 0.05))
-  (gr_line (start 221.99504 17.955629) (end 221.180001 19.142001) (layer "User.2") (width 0.05))
-  (gr_line (start 58.9 99.15) (end 110.5 99.15) (layer "User.2") (width 2.1))
-  (gr_line (start 189.500002 -17.099998) (end 190.820001 -23.319999) (layer "User.2") (width 0.05))
-  (gr_line (start 144.751903 102.301903) (end 134 102.3) (layer "User.2") (width 2.1))
-  (gr_line (start 144.751903 71.198097) (end 134 71.2) (layer "User.2") (width 2.1))
-  (gr_line (start 72.925951 102.300952) (end 62.174048 102.302855) (layer "User.2") (width 2.1))
-  (gr_line (start 72.925951 71.200952) (end 62.174048 71.199049) (layer "User.2") (width 2.1))
-  (gr_arc (start 148.001903 99.051903) (mid 147.05 101.35) (end 144.751903 102.301903) (layer "User.2") (width 2.1))
-  (gr_line (start 190.000001 17.950001) (end 190.820001 19.142001) (layer "User.2") (width 0.05))
-  (gr_line (start 189.495041 11.994372) (end 190.000001 14.390001) (layer "User.2") (width 0.05))
-  (gr_arc (start 222.504961 -17.09437) (mid 227.999403 -2.546248) (end 222.5 12) (layer "User.2") (width 0.05))
-  (gr_arc (start 144.751903 71.198097) (mid 147.05 72.15) (end 148.001903 74.448097) (layer "User.2") (width 2.1))
-  (gr_line (start 222.504961 -17.09437) (end 221.190001 -23.319999) (layer "User.2") (width 0.05))
-  (gr_arc (start 62.174048 102.302855) (mid 59.875951 101.350952) (end 58.924048 99.052855) (layer "User.2") (width 2.1))
-  (gr_line (start 190.820001 -23.319999) (end 221.190001 -23.319999) (layer "User.2") (width 0.05))
-  (gr_arc (start 58.924048 74.449049) (mid 59.875951 72.150952) (end 62.174048 71.199049) (layer "User.2") (width 2.1))
-  (gr_line (start 221.99504 14.395629) (end 221.99504 17.955629) (layer "User.2") (width 0.05))
-  (gr_arc (start 189.495041 11.994372) (mid 184.000599 -2.55375) (end 189.500002 -17.099998) (layer "User.2") (width 0.05))
-  (gr_line (start 190.820001 19.142001) (end 221.180001 19.142001) (layer "User.2") (width 0.05))
   (gr_line (start 83 159.5) (end 79 159.5) (layer "User.4") (width 0.15))
   (gr_line (start 106 30.5) (end 106 191) (layer "User.4") (width 0.15))
@@
   (segment (start 82.473945 80.076055) (end 85.898945 83.501055) (width 0.25) (layer "B.Cu") (net 53))
   (segment (start 81.85 76.65) (end 81.55 76.65) (width 0.25) (layer "B.Cu") (net 53))
-  (segment (start 86.8875 77.1) (end 86.4 77.1) (width 0.25) (layer "B.Cu") (net 53))
   (segment (start 82.2 77) (end 81.85 76.65) (width 0.25) (layer "B.Cu") (net 53))
   (segment (start 90.7 88.45) (end 90.7 88.30211) (width 0.25) (layer "B.Cu") (net 53))
@@
     )
   )
-  (group "" (id ff551455-fbe6-45f5-b1dd-91d405accebb)
-    (members
-      1b14a23a-a1e4-4f61-b7c6-ed0f52a809c1
-      1ddab5eb-e355-469b-8382-fc57ea75c27a
-      1e50f4bc-24a9-4da1-bfb5-9ae390963a14
-      29c517f6-bcc5-4a68-ad53-dcb33de48db9
-      9150e88d-e647-47d7-8b8b-7099f59ebb52
-      92ad17d0-1bbe-434a-af22-0a320c286e44
-      9e001289-b936-4c76-ad10-7aa978561df4
-      a16208a9-1a00-4e65-874a-d0f932b96a76
-      d1925e5c-8005-48e1-a460-7d2e97cff458
-      ee163c32-bc42-47b4-9428-9d74779c3f68
-      f592e097-2720-4c13-be2f-94373f3c272e
-      fad7dc67-05ed-4bec-8b90-20ba95187395
-    )
-  )
